File: eSimLibrary/2bit_DAC/2bit_DAC.sch (KiCad schematic (older format))
At the start: 5 parts, among them U1 PORT

Commit message: update
Parts:
- removed U?: PORT, symbol PORT
- added unit 7 of U1
Connections:
- net vout: now also U1.6; no longer U1.5
- net vrefl: now also U1.5
- net at S1.7 (din_buf): now also U1.7; no longer U1.6
Changed lines of the file:
@@
 $Comp
 L PORT U1
-U 4 1 643E4B11
+U 4 1 6443CD00
 P 4750 2300
 F 0 "U1" H 4800 2400 30  0000 C CNN
@@
 $Comp
 L resistor R1
-U 1 1 643E4A8A
+U 1 1 6443CD01
 P 4700 2800
 F 0 "R1" H 4750 2930 50  0000 C CNN
@@
 $Comp
 L switch_2n S1
-U 1 1 6443803F
+U 1 1 6443CD02
 P 4650 3950
 F 0 "S1" H 5350 3100 60  0000 C CNN
@@
 $Comp
 L PORT U1
-U 2 1 6443832D
+U 2 1 6443CD03
 P 3300 3900
 F 0 "U1" H 3350 4000 30  0000 C CNN
@@
 $Comp
 L switch S2
-U 1 1 6443C8B2
+U 1 1 6443CD04
 P 6950 4050
 F 0 "S2" H 6600 3750 60  0000 C CNN
@@
 $Comp
 L PORT U1
-U 3 1 6443C967
+U 3 1 6443CD05
 P 6000 4000
 F 0 "U1" H 6050 4100 30  0000 C CNN
@@
 $Comp
 L PORT U1
-U 1 1 6443C9AC
+U 1 1 6443CD06
 P 6300 2500
 F 0 "U1" H 6350 2600 30  0000 C CNN
@@
 $Comp
 L PORT U1
-U 5 1 6443CA76
+U 6 1 6443CD07
 P 7950 4050
 F 0 "U1" H 8000 4150 30  0000 C CNN
@@
 F 2 "" H 7950 4050 60  0000 C CNN
 F 3 "" H 7950 4050 60  0000 C CNN
-	5    7950 4050
+	6    7950 4050
 	-1   0    0    1
 $EndComp
@@
 $Comp
 L PORT U1
-U 6 1 6443CD41
+U 7 1 6443CD08
 P 6000 4600
 F 0 "U1" H 6050 4700 30  0000 C CNN
@@
 F 2 "" H 6000 4600 60  0000 C CNN
 F 3 "" H 6000 4600 60  0000 C CNN
-	6    6000 4600
+	7    6000 4600
 	-1   0    0    1
 $EndComp
@@
 vrefl
 $Comp
-L PORT U?
-U 7 1 6443D6A0
+L PORT U1
+U 5 1 6443CD09
 P 4750 5600
-F 0 "U?" H 4800 5700 30  0000 C CNN
+F 0 "U1" H 4800 5700 30  0000 C CNN
 F 1 "PORT" H 4750 5600 30  0000 C CNN
 F 2 "" H 4750 5600 60  0000 C CNN
 F 3 "" H 4750 5600 60  0000 C CNN
-	7    4750 5600
+	5    4750 5600
 	0    -1   -1   0
 $EndComp

Commit message: update
Parts:
- added unit 8 of U1
Connections:
- net d0: now also U1.4; no longer U1.2
- net d1: now also U1.5; no longer U1.3
- net vrefh: now also U1.2; no longer U1.4
- net vrefl: now also U1.3; no longer U1.5
- net d1_buf: now reaches S2.6 (Dx_buf)
- net d1_buf: now also U1.8
Changed lines of the file:
@@
 $Comp
 L PORT U1
-U 4 1 6443CD00
+U 2 1 6443CD00
 P 4750 2300
 F 0 "U1" H 4800 2400 30  0000 C CNN
@@
 F 2 "" H 4750 2300 60  0000 C CNN
 F 3 "" H 4750 2300 60  0000 C CNN
-	4    4750 2300
+	2    4750 2300
 	0    1    1    0
 $EndComp
@@
 $Comp
 L PORT U1
-U 2 1 6443CD03
+U 4 1 6443CD03
 P 3300 3900
 F 0 "U1" H 3350 4000 30  0000 C CNN
@@
 F 2 "" H 3300 3900 60  0000 C CNN
 F 3 "" H 3300 3900 60  0000 C CNN
-	2    3300 3900
+	4    3300 3900
 	1    0    0    -1
 $EndComp
@@
 $Comp
 L PORT U1
-U 3 1 6443CD05
+U 5 1 6443CD05
 P 6000 4000
 F 0 "U1" H 6050 4100 30  0000 C CNN
@@
 F 2 "" H 6000 4000 60  0000 C CNN
 F 3 "" H 6000 4000 60  0000 C CNN
-	3    6000 4000
+	5    6000 4000
 	1    0    0    -1
 $EndComp
@@
 	-1   0    0    1
 $EndComp
-Text Label 5600 4600 0    60   ~ 0
-d0_buf
 Wire Wire Line
 	4750 2550 4750 2700
@@
 	7700 4050 7500 4050
 Wire Wire Line
-	5750 4600 5650 4600
-Wire Wire Line
 	4750 4900 4750 5350
 Text Label 4750 5050 0    60   ~ 0
@@
 $Comp
 L PORT U1
-U 5 1 6443CD09
+U 3 1 6443CD09
 P 4750 5600
 F 0 "U1" H 4800 5700 30  0000 C CNN
@@
 F 2 "" H 4750 5600 60  0000 C CNN
 F 3 "" H 4750 5600 60  0000 C CNN
-	5    4750 5600
+	3    4750 5600
 	0    -1   -1   0
 $EndComp
+$Comp
+L PORT U1
+U 8 1 644BA539
+P 7950 4200
+F 0 "U1" H 8000 4300 30  0000 C CNN
+F 1 "PORT" H 7950 4200 30  0000 C CNN
+F 2 "" H 7950 4200 60  0000 C CNN
+F 3 "" H 7950 4200 60  0000 C CNN
+	8    7950 4200
+	-1   0    0    1
+$EndComp
+Wire Wire Line
+	7700 4200 7500 4200
+Text Label 7500 4200 0    60   ~ 0
+d1_buf
+Text Label 5600 4600 0    60   ~ 0
+d0_buf
+Wire Wire Line
+	5750 4600 5650 4600
 $EndSCHEMATC
