File: eSimLibrary/switch/switch.sch (KiCad schematic (older format))
At the start: 9 parts, among them M1 mosfet_n, M2 mosfet_p, M3 mosfet_n, M4 mosfet_p, M5 mosfet_n, M6 mosfet_p, M7 mosfet_p, M8 mosfet_n, U1 PORT

Commit message: update
Parts:
- added unit 6 of U1
Connections:
- net vrefh: now also U1.2; no longer U1.3
- net vrefl: now also U1.3; no longer U1.4
- net Dx_buf: now reaches M5.1 (D), M6.1 (D), M7.2 (G), M8.2 (G)
- net Dx_buf: now also U1.6
- net digital_input renamed Dx
- net Dx: now also U1.4; no longer U1.2
Changed lines of the file:
@@
 $Comp
 L mosfet_p M6
-U 1 1 643E446D
+U 1 1 644B9D83
 P 5350 3000
 F 0 "M6" H 5300 3050 50  0000 R CNN
@@
 $Comp
 L mosfet_n M5
-U 1 1 643E446E
+U 1 1 644B9D84
 P 5300 3450
 F 0 "M5" H 5300 3300 50  0000 R CNN
@@
 	1    0    0    -1
 $EndComp
-$Comp
-L GND #PWR3
-U 1 1 643E446F
+Entry Wire Line
+	5300 3450 5400 3550
+$Comp
+L GND #PWR01
+U 1 1 644B9D85
 P 5500 4100
-F 0 "#PWR3" H 5500 3850 50  0001 C CNN
+F 0 "#PWR01" H 5500 3850 50  0001 C CNN
 F 1 "GND" H 5500 3950 50  0000 C CNN
 F 2 "" H 5500 4100 50  0001 C CNN
@@
 $Comp
 L mosfet_p M2
-U 1 1 643E4470
+U 1 1 644B9D86
 P 3800 3000
 F 0 "M2" H 3750 3050 50  0000 R CNN
@@
 $Comp
 L mosfet_n M1
-U 1 1 643E4471
+U 1 1 644B9D87
 P 3750 3450
 F 0 "M1" H 3750 3300 50  0000 R CNN
@@
 $EndComp
 $Comp
-L GND #PWR1
-U 1 1 643E4472
+L GND #PWR02
+U 1 1 644B9D88
 P 3950 4100
-F 0 "#PWR1" H 3950 3850 50  0001 C CNN
+F 0 "#PWR02" H 3950 3850 50  0001 C CNN
 F 1 "GND" H 3950 3950 50  0000 C CNN
 F 2 "" H 3950 4100 50  0001 C CNN
@@
 $Comp
 L mosfet_n M3
-U 1 1 643E4473
+U 1 1 644B9D89
 P 5050 5450
 F 0 "M3" H 5050 5300 50  0000 R CNN
@@
 $Comp
 L mosfet_p M4
-U 1 1 643E4474
+U 1 1 644B9D8A
 P 5100 4850
 F 0 "M4" H 5050 4900 50  0000 R CNN
@@
 $Comp
 L mosfet_n M8
-U 1 1 643E4475
+U 1 1 644B9D8B
 P 6500 4650
 F 0 "M8" H 6500 4500 50  0000 R CNN
@@
 $Comp
 L mosfet_p M7
-U 1 1 643E4476
+U 1 1 644B9D8C
 P 6450 5600
 F 0 "M7" H 6400 5650 50  0000 R CNN
@@
 $EndComp
 $Comp
-L GND #PWR2
-U 1 1 643E4477
+L GND #PWR03
+U 1 1 644B9D8D
 P 5350 5800
-F 0 "#PWR2" H 5350 5550 50  0001 C CNN
+F 0 "#PWR03" H 5350 5550 50  0001 C CNN
 F 1 "GND" H 5350 5650 50  0000 C CNN
 F 2 "" H 5350 5800 50  0001 C CNN
@@
 $Comp
 L PORT U1
-U 1 1 643E4478
+U 1 1 644B9D8E
 P 4800 2200
 F 0 "U1" H 4850 2300 30  0000 C CNN
@@
 $Comp
 L PORT U1
-U 2 1 643E4479
+U 4 1 644B9D8F
 P 2650 3300
 F 0 "U1" H 2700 3400 30  0000 C CNN
@@
 F 2 "" H 2650 3300 60  0000 C CNN
 F 3 "" H 2650 3300 60  0000 C CNN
-	2    2650 3300
-	1    0    0    -1
-$EndComp
-$Comp
-L PORT U1
-U 3 1 643E447A
+	4    2650 3300
+	1    0    0    -1
+$EndComp
+$Comp
+L PORT U1
+U 2 1 644B9D90
 P 5800 4200
 F 0 "U1" H 5850 4300 30  0000 C CNN
@@
 F 2 "" H 5800 4200 60  0000 C CNN
 F 3 "" H 5800 4200 60  0000 C CNN
-	3    5800 4200
+	2    5800 4200
 	0    1    1    0
 $EndComp
 $Comp
 L PORT U1
-U 4 1 643E447B
+U 3 1 644B9D91
 P 5800 6400
 F 0 "U1" H 5850 6500 30  0000 C CNN
@@
 F 2 "" H 5800 6400 60  0000 C CNN
 F 3 "" H 5800 6400 60  0000 C CNN
-	4    5800 6400
+	3    5800 6400
 	0    -1   -1   0
 $EndComp
 $Comp
 L PORT U1
-U 5 1 643E447C
+U 5 1 644B9D92
 P 5800 5600
 F 0 "U1" H 5850 5700 30  0000 C CNN
@@
 Wire Wire Line
 	5500 3200 5500 3450
+Text Label 4850 2550 0    60   ~ 0
+vdd
 Text Label 5700 5250 0    60   ~ 0
 Vout
@@
 Text Label 5850 6050 0    60   ~ 0
 vrefl
-$Comp
-L GND #PWR4
-U 1 1 643E447D
+Text Label 5350 4700 0    60   ~ 0
+vdd
+Text Label 6200 5450 0    60   ~ 0
+vdd
+$Comp
+L GND #PWR04
+U 1 1 644B9D93
 P 6200 5100
-F 0 "#PWR4" H 6200 4850 50  0001 C CNN
+F 0 "#PWR04" H 6200 4850 50  0001 C CNN
 F 1 "GND" H 6200 4950 50  0000 C CNN
 F 2 "" H 6200 5100 50  0001 C CNN
@@
 	6200 5100 6200 5000
 $Comp
-L PWR_FLAG #FLG1
-U 1 1 643E447E
+L PWR_FLAG #FLG05
+U 1 1 644B9D94
 P 6050 5000
-F 0 "#FLG1" H 6050 5075 50  0001 C CNN
+F 0 "#FLG05" H 6050 5075 50  0001 C CNN
 F 1 "PWR_FLAG" H 6050 5150 50  0000 C CNN
 F 2 "" H 6050 5000 50  0001 C CNN
@@
 Connection ~ 6200 5000
 Text Label 2900 3300 0    60   ~ 0
-digital_input
-Text Label 4850 2550 0    60   ~ 0
-vdd
-Text Label 5350 4700 0    60   ~ 0
-vdd
-Text Label 6200 5450 0    60   ~ 0
-vdd
+Dx
+$Comp
+L PORT U1
+U 6 1 644B9D95
+P 7900 4150
+F 0 "U1" H 7950 4250 30  0000 C CNN
+F 1 "PORT" H 7900 4150 30  0000 C CNN
+F 2 "" H 7900 4150 60  0000 C CNN
+F 3 "" H 7900 4150 60  0000 C CNN
+	6    7900 4150
+	-1   0    0    1
+$EndComp
+Wire Wire Line
+	7650 4150 7550 4150
+Connection ~ 7550 4150
+Text Label 7100 3300 0    60   ~ 0
+Dx_buf
 $EndSCHEMATC
