File: eSimLibrary/switch_2n/switch_2n.sch (KiCad schematic (older format))
At the start: 3 parts

Commit message: update
Parts:
- removed R?: resistor, symbol resistor
- removed S?: switch_2n, symbol switch_2n
- removed S?: switch, symbol switch
- added M? (x6): mosfet_p, symbol mosfet_p
- added M? (x6): mosfet_n, symbol mosfet_n
- added R? (x3): resistor, symbol resistor
- added U1: PORT, symbol PORT
Connections:
- net labels added: Dx, Dx_buf, GND, vdd, vin_1, vinh_2, vinl, vinl_2, vouth, voutl, vrefh, vrefl
- wire segments 1 -> 90
