File: schematics/switch_2n/switch_2n.sch (KiCad schematic (older format))
At the start: 17 parts, among them M1 mosfet_p, M10 mosfet_p, M11 mosfet_p, M12 mosfet_n, M2 mosfet_n, M3 mosfet_p, M4 mosfet_n, M5 mosfet_p, M6 mosfet_n, M7 mosfet_n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

Commit message: update
Parts:
- renumbered U2 to U1
Connections:
- net vinh: now also U1.2; no longer U1.1
- net vinl: now also U1.3; no longer U1.2
- net vouth: now also U1.5; no longer U1.4
- net voutl: now also U1.6; no longer U1.5
- net din renamed Dx
- net Dx: now also U1.4; no longer U1.2
- net din_buf renamed Dx_buf
- net Dx_buf: now also U1.8; no longer U1.3
Changed lines of the file:
@@
 LIBS:eSim_SKY130
 LIBS:eSim_SKY130_Subckts
+LIBS:switch_2n-cache
 EELAYER 25 0
 EELAYER END
@@
 $Comp
 L PORT U1
-U 2 1 643BDA30
+U 4 1 643BDA30
 P 2050 2450
 F 0 "U1" H 2100 2550 30  0000 C CNN
@@
 F 2 "" H 2050 2450 60  0000 C CNN
 F 3 "" H 2050 2450 60  0000 C CNN
-	2    2050 2450
-	1    0    0    -1
-$EndComp
-$Comp
-L PORT U1
-U 5 1 643BE0A2
+	4    2050 2450
+	1    0    0    -1
+$EndComp
+$Comp
+L PORT U1
+U 6 1 643BE0A2
 P 5200 4750
 F 0 "U1" H 5250 4850 30  0000 C CNN
@@
 F 2 "" H 5200 4750 60  0000 C CNN
 F 3 "" H 5200 4750 60  0000 C CNN
-	5    5200 4750
+	6    5200 4750
 	0    -1   -1   0
 $EndComp
@@
 Connection ~ 5600 4150
 Text Label 2300 2450 0    60   ~ 0
-din
+Dx
 $Comp
 L mosfet_p M10
@@
 vouth
 $Comp
-L PORT U2
-U 4 1 644298D6
+L PORT U1
+U 5 1 644298D6
 P 8600 4750
-F 0 "U2" H 8650 4850 30  0000 C CNN
+F 0 "U1" H 8650 4850 30  0000 C CNN
 F 1 "PORT" H 8600 4750 30  0000 C CNN
 F 2 "" H 8600 4750 60  0000 C CNN
 F 3 "" H 8600 4750 60  0000 C CNN
-	4    8600 4750
+	5    8600 4750
 	0    -1   -1   0
 $EndComp
@@
 vinh_2
 Text Label 7900 3050 0    60   ~ 0
-din_buf
-$Comp
-L PORT U2
-U 3 1 6442A70A
+Dx_buf
+$Comp
+L PORT U1
+U 8 1 6442A70A
 P 7800 2700
-F 0 "U2" H 7850 2800 30  0000 C CNN
+F 0 "U1" H 7850 2800 30  0000 C CNN
 F 1 "PORT" H 7800 2700 30  0000 C CNN
 F 2 "" H 7800 2700 60  0000 C CNN
 F 3 "" H 7800 2700 60  0000 C CNN
-	3    7800 2700
+	8    7800 2700
 	0    1    1    0
 $EndComp
@@
 	1950 4550 1950 5150
 $Comp
-L PORT U2
-U 2 1 6442B0A6
+L PORT U1
+U 3 1 6442B0A6
 P 1950 6000
-F 0 "U2" H 2000 6100 30  0000 C CNN
+F 0 "U1" H 2000 6100 30  0000 C CNN
 F 1 "PORT" H 1950 6000 30  0000 C CNN
 F 2 "" H 1950 6000 60  0000 C CNN
 F 3 "" H 1950 6000 60  0000 C CNN
-	2    1950 6000
+	3    1950 6000
 	0    -1   -1   0
 $EndComp
@@
 	1950 3350 1950 3600
 $Comp
-L PORT U2
-U 1 1 6442B471
+L PORT U1
+U 2 1 6442B471
 P 1950 3100
-F 0 "U2" H 2000 3200 30  0000 C CNN
+F 0 "U1" H 2000 3200 30  0000 C CNN
 F 1 "PORT" H 1950 3100 30  0000 C CNN
 F 2 "" H 1950 3100 60  0000 C CNN
 F 3 "" H 1950 3100 60  0000 C CNN
-	1    1950 3100
+	2    1950 3100
 	0    1    1    0
 $EndComp
