File: schematics/switch/switch.sch (KiCad schematic (older format))
At the start: 9 parts, among them M1 mosfet_p, M2 mosfet_n, M3 mosfet_p, M4 mosfet_n, M5 mosfet_p, M6 mosfet_n, M7 mosfet_n, M8 mosfet_p, U1 PORT

Commit message: update
Parts:
- added unit 6 of U1
Connections:
- net Dx_buf: now reaches M3.1 (D), M4.1 (D), M7.2 (G), M8.2 (G)
- net Dx_buf: now also U1.6
- net digital_input renamed Dx
Changed lines of the file:
@@
 LIBS:eSim_Nghdl
 LIBS:eSim_Ngveri
+LIBS:switch-cache
 EELAYER 25 0
 EELAYER END
@@
 Connection ~ 6200 5000
 Text Label 2900 3300 0    60   ~ 0
-digital_input
+Dx
+$Comp
+L PORT U1
+U 6 1 644B99EE
+P 7900 4150
+F 0 "U1" H 7950 4250 30  0000 C CNN
+F 1 "PORT" H 7900 4150 30  0000 C CNN
+F 2 "" H 7900 4150 60  0000 C CNN
+F 3 "" H 7900 4150 60  0000 C CNN
+	6    7900 4150
+	-1   0    0    1
+$EndComp
+Wire Wire Line
+	7650 4150 7550 4150
+Connection ~ 7550 4150
+Text Label 7100 3300 0    60   ~ 0
+Dx_buf
 $EndSCHEMATC

Commit message: update
Changed lines of the file:
@@
 	1    0    0    -1
 $EndComp
-Entry Wire Line
-	5300 3450 5400 3550
 $Comp
 L GND #PWR01
